File: water/test/test.kicad_pcb (KiCad board)
At the start: 2 copper layers, 100 x 67.5 mm, 121 parts, among them J1 HEADER_1X6, J2 term_block_4-pin, J3 term_block_4-pin, J4 term_block_4-pin, J5 term_block_4-pin, M1 MNT-3MM, M2 MNT-3MM, M3 MNT-3MM, M4 MNT-3MM, Q1 MOSFET-N, Q2 MOSFET-N, Q3 MOSFET-N, Q4 MOSFET-N, Q5 MOSFET-N, U1 MPX5100, U10 Level_Shifter_single, U11 Level_Shifter_single, U12 Level_Shifter_single, U13 Relay-EC2-5NU, U14 Relay-EC2-5NU, U15 MC34063A_buck, U16 TLV1117_3.3V, U2 RS485_TRX_14pin, U3 PIC16F1829_SOIC, U4 Level_Shifter_single, U5 Level_Shifter_single, U6 Temp_SOT23-3, U7 23K256, U8 Level_Shifter_single, U9 Level_Shifter_single

Commit message: Not exactly sure what this all is, but committing it anyways
Changed lines of the file:
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@@
-(kicad_pcb (version 4) (host pcbnew 4.0.7)
+(kicad_pcb (version 20171130) (host pcbnew 5.0.0-fee4fd1~66~ubuntu18.04.1)
   (general
-    (links 250)
-    (no_connects 7)
-    (area 29.924999 102.424999 130.075001 170.075001)
     (thickness 1.6)
     (drawings 33)
@@
   (page A4)
   (layers
-    (0 F.Cu signal)
+    (0 F.Cu signal hide)
     (31 B.Cu signal)
     (32 B.Adhes user)
@@
     (aux_axis_origin 30 170)
     (grid_origin 30 170)
-    (visible_elements 7FFEEF7F)
+    (visible_elements 7FFF6D7F)
     (pcbplotparams
       (layerselection 0x010f0_80000001)
       (usegerberextensions true)
+      (usegerberattributes false)
+      (usegerberadvancedattributes false)
+      (creategerberjobfile false)
       (excludeedgelayer true)
       (linewidth 0.100000)
@@
       (hpglpennumber 1)
       (hpglpenspeed 20)
-      (hpglpendiameter 15)
-      (hpglpenoverlay 2)
+      (hpglpendiameter 15.000000)
       (psnegative false)
       (psa4output false)
@@
       (drillshape 0)
       (scaleselection 1)
-      (outputdirectory gerbers/))
+      (outputdirectory "gerbers/"))
   )
   (net 0 "")
@@
   (module ICs:SO-20_300 (layer F.Cu)
     (at 84.074 132.334 270)
-    (fp_text reference U3 (at -1.434 -7.226 360) (layer F.SilkS)
+    (fp_text reference U3 (at -1.434 -7.226) (layer F.SilkS)
       (effects (font (size 1 1) (thickness 0.15)))
     )
@@
   (module switches:EC2-5NU (layer F.Cu)
     (at 53.34 125.73 270)
-    (fp_text reference U13 (at -4.572 -5.842 360) (layer F.SilkS)
+    (fp_text reference U13 (at -4.572 -5.842) (layer F.SilkS)
       (effects (font (size 1 1) (thickness 0.15)))
     )
@@
   (module switches:EC2-5NU (layer F.Cu)
     (at 53.34 137.16 270)
-    (fp_text reference U14 (at -4.572 -6.096 360) (layer F.SilkS)
+    (fp_text reference U14 (at -4.572 -6.096) (layer F.SilkS)
       (effects (font (size 1 1) (thickness 0.15)))
     )
@@
     (effects (font (size 1 1) (thickness 0.2)))
   )
-  (gr_text GND (at 41.9 124.6 360) (layer F.SilkS)
+  (gr_text GND (at 41.9 124.6) (layer F.SilkS)
     (effects (font (size 1 1) (thickness 0.2)))
   )
-  (gr_text GND (at 42.1 134.6 360) (layer F.SilkS)
+  (gr_text GND (at 42.1 134.6) (layer F.SilkS)
     (effects (font (size 1 1) (thickness 0.2)))
   )
@@
     (effects (font (size 1 1) (thickness 0.2)))
   )
-  (gr_text GND (at 41.6 145.2 360) (layer F.SilkS)
+  (gr_text GND (at 41.6 145.2) (layer F.SilkS)
     (effects (font (size 1 1) (thickness 0.2)))
   )
