File: water/test/test.sch (KiCad schematic (older format))
At the start: 98 parts, among them J1 HEADER_1X6, J2 term_block_4-pin, J3 term_block_4-pin, J4 term_block_4-pin, J5 term_block_4-pin, M1 MNT-3MM, M2 MNT-3MM, M3 MNT-3MM, M4 MNT-3MM, Q1 MOSFET-N, Q2 MOSFET-N, Q3 MOSFET-N, Q4 MOSFET-N, Q5 MOSFET-N, U1 MPX5100, U10 Level_Shifter_single, U11 Level_Shifter_single, U12 Level_Shifter_single, U13 Relay-EC2-5NU, U14 Relay-EC2-5NU, U2 RS485_TRX_14pin, U3 PIC16F1829_SOIC, U4 Level_Shifter_single, U5 Level_Shifter_single, U6 Temp_SOT23-3, U7 23K256, U8 Level_Shifter_single, U9 Level_Shifter_single

Commit message: Not exactly sure what this all is, but committing it anyways
Parts:
- U1: symbol MPX5100 -> misc:MPX5100
Connections:
- wire segments 256 -> 277
Changed lines of the file:
@@
-EESchema Schematic File Version 2
-LIBS:connectors
-LIBS:diodes
-LIBS:mechanical
-LIBS:microchip_mcu
-LIBS:misc
-LIBS:passives
-LIBS:switches
-LIBS:transistors
-LIBS:IC_Interface
-LIBS:power
-LIBS:memory
-LIBS:regulators
+EESchema Schematic File Version 4
 LIBS:test-cache
-EELAYER 25 0
+EELAYER 26 0
 EELAYER END
 $Descr A4 11693 8268
@@
 nSPI_CS
 $Comp
-L MPX5100 U1
+L misc:MPX5100 U1
 U 1 1 5A190136
 P 1900 1050
@@
 $EndComp
 $Comp
-L +5V #PWR1
+L power:+5V #PWR1
 U 1 1 5A19FF4B
 P 800 950
@@
 	8450 1450 9450 1450
 Wire Wire Line
-	8100 1550 9450 1550
+	8100 1550 8200 1550
 Wire Wire Line
 	9300 1750 9300 1850
@@
 Connection ~ 8200 1550
 Wire Wire Line
-	9300 2200 9300 2300
+	9300 2200 9300 2250
 Wire Wire Line
 	9300 2250 9450 2250
@@
 	5100 1100 5100 900
 Wire Wire Line
-	5000 900  5200 900
+	5000 900  5100 900
 Wire Wire Line
 	5550 900  5650 900
@@
 	9300 2800 8800 2800
 Wire Wire Line
-	8800 2700 8800 2900
+	8800 2700 8800 2800
 Wire Wire Line
 	10350 2800 10250 2800
 Wire Wire Line
-	2450 3750 2900 3750
+	2450 3750 2550 3750
 Wire Wire Line
 	2550 3750 2550 3650
@@
 	1950 5700 2050 5700
 Wire Wire Line
-	1950 5050 1950 5700
+	1950 5050 1950 5200
 Wire Wire Line
 	2150 5450 1950 5450
 Connection ~ 1950 5450
 Wire Wire Line
-	2650 5700 2900 5700
+	2650 5700 2800 5700
 Wire Wire Line
 	2800 5700 2800 5450
 Wire Wire Line
-	2600 5450 2900 5450
+	2600 5450 2800 5450
 Connection ~ 2800 5700
 Wire Wire Line
@@
 	3900 6850 4000 6850
 Wire Wire Line
-	3900 6200 3900 6850
+	3900 6200 3900 6350
 Wire Wire Line
 	4100 6600 3900 6600
 Connection ~ 3900 6600
 Wire Wire Line
-	4600 6850 4850 6850
+	4600 6850 4750 6850
 Wire Wire Line
 	4750 6850 4750 6600
 Wire Wire Line
-	4550 6600 4850 6600
+	4550 6600 4750 6600
 Connection ~ 4750 6850
 Wire Wire Line
@@
 	4650 4050 4650 4000
 Wire Wire Line
-	4300 3550 4750 3550
+	4300 3550 4650 3550
 Wire Wire Line
 	4650 3650 4650 3550
@@
 	1100 1900 1700 1900
 Wire Wire Line
-	1700 1800 1700 2000
+	1700 1800 1700 1900
 Connection ~ 1700 1900
 Wire Wire Line
@@
 $EndComp
 Wire Wire Line
-	9100 2700 9300 2700
-Wire Wire Line
-	10250 2700 10400 2700
-Wire Wire Line
 	10250 2900 10850 2900
 $Comp
@@
 	-1   0    0    1
 $EndComp
-Connection ~ 9200 2700
 Wire Wire Line
 	8850 2700 8800 2700
@@
 	-1   0    0    1
 $EndComp
-Connection ~ 10350 2700
 $Comp
 L GND #PWR70
@@
 	9250 3400 8750 3400
 Wire Wire Line
-	8750 3300 8750 3500
+	8750 3300 8750 3400
 Wire Wire Line
 	10300 3400 10200 3400
-Wire Wire Line
-	9050 3300 9250 3300
-Wire Wire Line
-	10200 3300 10350 3300
 Wire Wire Line
 	10200 3500 10800 3500
@@
 	-1   0    0    1
 $EndComp
-Connection ~ 9150 3300
 Wire Wire Line
 	8800 3300 8750 3300
@@
 	-1   0    0    1
 $EndComp
-Connection ~ 10300 3300
 $Comp
 L GND #PWR66
@@
 	9250 4050 8550 4050
 Wire Wire Line
-	8550 3950 8550 4150
+	8550 3950 8550 4050
 Wire Wire Line
 	10300 4050 10200 4050
-Wire Wire Line
-	8850 3950 9250 3950
-Wire Wire Line
-	10200 3950 10350 3950
 Wire Wire Line
 	10200 4150 10800 4150
@@
 	-1   0    0    1
 $EndComp
-Connection ~ 9150 3950
 Wire Wire Line
 	8600 3950 8550 3950
@@
 	-1   0    0    1
 $EndComp
-Connection ~ 10300 3950
 $Comp
 L GND #PWR67
@@
 	9250 4700 8550 4700
 Wire Wire Line
-	8550 4600 8550 4800
+	8550 4600 8550 4700
 Wire Wire Line
 	10300 4700 10200 4700
-Wire Wire Line
-	8850 4600 9250 4600
-Wire Wire Line
-	10200 4600 10350 4600
 Wire Wire Line
 	10200 4800 10800 4800
@@
 	-1   0    0    1
 $EndComp
-Connection ~ 9150 4600
 Wire Wire Line
 	8600 4600 8550 4600
@@
 	-1   0    0    1
 $EndComp
-Connection ~ 10300 4600
 $Comp
 L GND #PWR68
@@
 	6250 5000 5550 5000
 Wire Wire Line
-	5550 4900 5550 5100
+	5550 4900 5550 5000
 Wire Wire Line
 	7300 5000 7200 5000
-Wire Wire Line
-	5850 4900 6250 4900
-Wire Wire Line
-	7200 4900 7350 4900
 Wire Wire Line
 	7200 5100 7800 5100
@@
 	-1   0    0    1
 $EndComp
-Connection ~ 6150 4900
 Wire Wire Line
 	5600 4900 5550 4900
@@
 	-1   0    0    1
 $EndComp
-Connection ~ 7300 4900
 $Comp
 L GND #PWR41
@@
 	9250 5350 8550 5350
 Wire Wire Line
-	8550 5250 8550 5450
+	8550 5250 8550 5350
 Wire Wire Line
 	10300 5350 10200 5350
-Wire Wire Line
-	8850 5250 9250 5250
-Wire Wire Line
-	10200 5250 10350 5250
 Wire Wire Line
 	10200 5450 10800 5450
@@
 	-1   0    0    1
 $EndComp
-Connection ~ 9150 5250
 Wire Wire Line
 	8600 5250 8550 5250
@@
 	-1   0    0    1
 $EndComp
-Connection ~ 10300 5250
 $Comp
 L GND #PWR69
@@
 	6250 5750 5550 5750
 Wire Wire Line
-	5550 5650 5550 5850
+	5550 5650 5550 5750
 Wire Wire Line
 	7300 5750 7200 5750
-Wire Wire Line
-	5850 5650 6250 5650
-Wire Wire Line
-	7200 5650 7350 5650
 Wire Wire Line
 	7200 5850 7800 5850
@@
 	-1   0    0    1
 $EndComp
-Connection ~ 6150 5650
 Wire Wire Line
 	5600 5650 5550 5650
@@
 	-1   0    0    1
 $EndComp
-Connection ~ 7300 5650
 $Comp
 L GND #PWR42
@@
 Text Notes 2250 1750 0    60   ~ 0
 RA5 is not analog
+Wire Wire Line
+	8200 1550 9450 1550
+Wire Wire Line
+	9300 2250 9300 2300
+Wire Wire Line
+	5100 900  5200 900
+Wire Wire Line
+	2550 3750 2900 3750
+Wire Wire Line
+	1950 5450 1950 5700
+Wire Wire Line
+	2800 5700 2900 5700
+Wire Wire Line
+	1950 5200 1950 5450
+Wire Wire Line
+	2800 5450 2900 5450
+Wire Wire Line
+	3900 6600 3900 6850
+Wire Wire Line
+	4750 6850 4850 6850
+Wire Wire Line
+	3900 6350 3900 6600
+Wire Wire Line
+	4750 6600 4850 6600
+Wire Wire Line
+	4650 3550 4750 3550
+Wire Wire Line
+	1700 1900 1700 2000
+Wire Wire Line
+	8800 2800 8800 2900
+Wire Wire Line
+	8750 3400 8750 3500
+Wire Wire Line
+	8550 4050 8550 4150
+Wire Wire Line
+	8550 4700 8550 4800
+Wire Wire Line
+	5550 5000 5550 5100
+Wire Wire Line
+	8550 5350 8550 5450
+Wire Wire Line
+	5550 5750 5550 5850
+Wire Wire Line
+	10250 2700 10400 2700
+Wire Wire Line
+	10200 3300 10350 3300
+Wire Wire Line
+	10200 3950 10350 3950
+Wire Wire Line
+	10200 4600 10350 4600
+Wire Wire Line
+	7200 4900 7350 4900
+Wire Wire Line
+	10200 5250 10350 5250
+Wire Wire Line
+	7200 5650 7350 5650
+Wire Wire Line
+	9100 2700 9300 2700
+Wire Wire Line
+	9050 3300 9250 3300
+Wire Wire Line
+	8850 3950 9250 3950
+Wire Wire Line
+	8850 4600 9250 4600
+Wire Wire Line
+	5850 4900 6250 4900
+Wire Wire Line
+	8850 5250 9250 5250
+Wire Wire Line
+	5850 5650 6250 5650
 $EndSCHEMATC
