File: sprinkler_nodes/_autosave-sprinkler_nodes.kicad_pcb (KiCad board)
At the start: 2 copper layers, 94 x 54.6 mm, 67 parts, among them J1 term_block_4-pin, J2 term_block_4-pin, J3 HEADER_1X6, Q1 NPN, Q2 NPN, U1 PIC16F1829_SOIC, U2 Temp_SOT23-3, U3 MP2456, U4 TLV1117_3.3V, U5 NC7SZ125, U6 MPX5100

Commit message: First shot of gerbers for sprinkler nodes
Routing:
- net +5V: vias 3 -> 2
Changed lines of the file:
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@@
     (thickness 1.6)
     (drawings 17)
-    (tracks 414)
+    (tracks 413)
     (zones 0)
     (modules 67)
@@
   (layers
     (0 F.Cu signal)
-    (31 B.Cu signal hide)
+    (31 B.Cu signal)
     (32 B.Adhes user)
     (33 F.Adhes user)
@@
     (visible_elements FFFDFF7F)
     (pcbplotparams
-      (layerselection 0x010fc_ffffffff)
+      (layerselection 0x010f0_ffffffff)
       (usegerberextensions false)
       (usegerberattributes false)
@@
       (psa4output false)
       (plotreference true)
-      (plotvalue true)
+      (plotvalue false)
       (plotinvisibletext false)
       (padsonsilk false)
@@
       (outputformat 1)
       (mirror false)
-      (drillshape 1)
+      (drillshape 0)
       (scaleselection 1)
-      (outputdirectory ""))
+      (outputdirectory "gerbers/"))
   )
   (net 0 "")
@@
   (segment (start 95.211 63.249) (end 93.69 64.77) (width 0.508) (layer F.Cu) (net 6) (status 800000))
   (segment (start 79.502 47.943) (end 80.3524 47.943) (width 0.254) (layer F.Cu) (net 6) (status 400000))
-  (via (at 80.3656 47.9298) (size 0.6096) (drill 0.3048) (layers F.Cu B.Cu) (net 6))
   (segment (start 80.3524 47.943) (end 80.3656 47.9298) (width 0.254) (layer F.Cu) (net 6))
   (segment (start 80.3656 47.9298) (end 80.8522 47.9298) (width 0.254) (layer F.Cu) (net 6))
