File: sprinkler_nodes/power.sch (KiCad schematic (older format))
At the start: 19 parts, among them U3 MP2456, U4 TLV1117_3.3V

Commit message: Updated part numbers
Parts:
- C5: MFG_PN {PN} -> UCM1H470MCL1GS
- D3: MFG_PN {PN} -> DFLS160-7
- D5: MFG_PN {PN} -> BAS16HT1G
- L1: MFG_PN {PN} -> CLF5030NIT-100M-D
- U4: symbol LDOs:TLV1117_3.3V -> regulators:TLV1117_3.3V; MFG_PN (none) -> TLV1117-33CDCYR
Changed lines of the file:
@@
 F 2 "diodes:SOD123" H 4850 1950 60  0001 C CNN
 F 3 "" H 4600 1950 60  0000 C CNN
-F 4 "{PN}" H 4700 2050 60  0001 C CNN "MFG_PN"
+F 4 "DFLS160-7" H 4700 2050 60  0001 C CNN "MFG_PN"
 	1    4750 2000
 	-1   0    0    1
@@
 F 4 "+" V 3400 4050 30  0000 L CNN "Polarity"
 F 5 "47uF" V 3550 4100 39  0000 L CNN "val"
-F 6 "{PN}" H 3600 4300 60  0001 C CNN "MFG_PN"
+F 6 "UCM1H470MCL1GS" H 3600 4300 60  0001 C CNN "MFG_PN"
 	1    3250 4050
 	0    1    1    0
@@
 F 3 "" H 5400 1850 60  0001 C CNN
 F 4 "10uH" H 5550 1684 40  0000 C CNN "val"
-F 5 "{PN}" H 5600 2050 60  0001 C CNN "MFG_PN"
+F 5 "CLF5030NIT-100M-D" H 5600 2050 60  0001 C CNN "MFG_PN"
 	1    5250 1800
 	-1   0    0    1
 $EndComp
 $Comp
-L LDOs:TLV1117_3.3V U?
+L regulators:TLV1117_3.3V U?
 U 1 1 5A19F674
 P 8050 2200
@@
 F 2 "ICs:SOT-223" H 8500 1850 60  0001 C CNN
 F 3 "" H 8050 2200 60  0000 C CNN
+F 4 "TLV1117-33CDCYR" H 0   0   50  0001 C CNN "MFG_PN"
 	1    8050 2200
 	1    0    0    -1
@@
 F 2 "diodes:SOD323" H 8400 1800 60  0001 C CNN
 F 3 "" H 8150 1800 60  0000 C CNN
-F 4 "{PN}" H 8250 1900 40  0001 C CNN "MFG_PN"
+F 4 "BAS16HT1G" H 8250 1900 40  0001 C CNN "MFG_PN"
 	1    8300 1850
 	-1   0    0    1
