File: sprinkler_nodes/sprinkler_nodes.sch (KiCad schematic (older format))
At the start: 22 parts, among them J1 term_block_4-pin, J2 term_block_4-pin, J3 HEADER_1X6, U1 PIC16F1829_SOIC, U2 Temp_SOT23-3, U6 MPX5100

Commit message: Rev 1.1 Sprinkler Nodes. Added more options for turning on valves
Parts:
- added C19, C20: CAP_0603, C0603, symbol passives:CAP_0603
- added Q3: Triac, ICs:Triode SMB-3, symbol transistors:Triac
- added R24, R25, R26, R27, R28, R29, R3, R30, R31, R32, R4: RES_0603, passives:R0603, symbol passives:RES_0603
Connections:
- net labels added: LOAD, TRIAC_G
- net labels removed: SW_24V_1
- wire segments 88 -> 125
Other:
- note added: "DNF"

Commit message: Updated part numbers
Parts:
- D2: MFG_PN {PN} -> DFLS160-7
- R30: MFG_PN RC0603JR-07470RL -> {PN}
- U6: MFG_PN (none) -> MPXV5100DP
Changed lines of the file:
@@
 F 2 "diodes:SOD123" H 8650 1000 60  0001 C CNN
 F 3 "" H 8400 1000 60  0000 C CNN
-F 4 "{PN}" H 8500 1100 60  0001 C CNN "MFG_PN"
+F 4 "DFLS160-7" H 8500 1100 60  0001 C CNN "MFG_PN"
 	1    8550 1050
 	-1   0    0    1
@@
 F 2 "ICs:MPX5100" H 6200 3400 60  0001 C CNN
 F 3 "" H 6250 3400 60  0001 C CNN
+F 4 "MPXV5100DP" H 0   0   50  0001 C CNN "MFG_PN"
 	1    6250 3400
 	1    0    0    -1
@@
 F 3 "" H 4050 1350 60  0000 C CNN
 F 4 "39" H 4250 1550 40  0000 C CNN "val"
-F 5 "RC0603JR-07470RL" H 4250 1500 60  0001 C CNN "MFG_PN"
+F 5 "{PN}" H 4250 1500 60  0001 C CNN "MFG_PN"
 	1    4250 1500
 	0    -1   -1   0
