File: sprinkler_nodes/transceiver.sch (KiCad schematic (older format))
At the start: 26 parts, among them Q1 NPN, Q2 NPN, U5 NC7SZ125

Commit message: Updated part numbers
Parts:
- D10: MFG_PN {PN} -> BAS16HT1G
- D11, D8: MFG_PN {PN} -> NSR0530HT1G
- D7, D9: MFG_PN {PN} -> DF2B7AE,H3F
Changed lines of the file:
@@
 F 2 "diodes:SOD323" H 3650 6500 60  0001 C CNN
 F 3 "" H 3400 6500 60  0000 C CNN
-F 4 "{PN}" H 3500 6600 60  0001 C CNN "MFG_PN"
+F 4 "DF2B7AE,H3F" H 3500 6600 60  0001 C CNN "MFG_PN"
 	1    3550 6550
 	-1   0    0    1
@@
 F 2 "diodes:SOD323" H 2450 3500 60  0001 C CNN
 F 3 "" H 2200 3500 60  0000 C CNN
-F 4 "{PN}" H 2300 3600 60  0001 C CNN "MFG_PN"
+F 4 "DF2B7AE,H3F" H 2300 3600 60  0001 C CNN "MFG_PN"
 	1    2350 3550
 	0    -1   -1   0
@@
 F 2 "diodes:SOD323" H 2850 3500 60  0001 C CNN
 F 3 "" H 2600 3500 60  0000 C CNN
-F 4 "{PN}" H 2700 3600 60  0001 C CNN "MFG_PN"
+F 4 "NSR0530HT1G" H 2700 3600 60  0001 C CNN "MFG_PN"
 	1    2750 3550
 	0    -1   -1   0
@@
 F 2 "diodes:SOD323" H 4300 3500 60  0001 C CNN
 F 3 "" H 4050 3500 60  0000 C CNN
-F 4 "{PN}" H 4150 3600 40  0001 C CNN "MFG_PN"
+F 4 "BAS16HT1G" H 4150 3600 40  0001 C CNN "MFG_PN"
 	1    4200 3550
 	1    0    0    -1
@@
 F 2 "diodes:SOD323" H 5450 3750 60  0001 C CNN
 F 3 "" H 5200 3750 60  0000 C CNN
-F 4 "{PN}" H 5300 3850 60  0001 C CNN "MFG_PN"
+F 4 "NSR0530HT1G" H 5300 3850 60  0001 C CNN "MFG_PN"
 	1    5350 3800
 	0    -1   -1   0
