File: sprinkler_node_buffer/sprinkler_node_buffer.sch (KiCad schematic (older format))
At the start: 11 parts

Commit message: Added sprinkler node buffer
Parts:
- removed BR?: MD5S_Diode_Bridge, diodes:MD5S, symbol diodes:MD5S_Diode_Bridge
- removed C?: CAP_ELEC, symbol passives:CAP_ELEC
- removed C? (x2): CAP_0805, C0805, symbol passives:CAP_0805
- removed D?: Zener_SOD123, diodes:SOD123, symbol diodes:Zener_SOD123
- removed D?: Diode_SOD123, diodes:SOD123, symbol diodes:Diode_SOD123
- removed Q?: NPN, ICs:SOT-23-3, symbol transistors:NPN
- removed R? (x2): RES_0603, R0603, symbol passives:RES_0603
- added C1, C2, C3, C4, C5, C6, C7, C8: CAP_0603, C0603, symbol passives:CAP_0603
- added D1, D2, D3, D4: Zener_SOD123, diodes:SOD123, symbol diodes:Zener_SOD123
- added Q1: NPN, ICs:SOT-23-3, symbol transistors:NPN
- added R1, R2, R3, R4, R5, R6, R7, R8, R9: RES_0603, R0603, symbol passives:RES_0603
- added U1, U2: NC7SZ125, ICs:SOT-23-5, symbol ICs:NC7SZ125
- gave numbers to parts that had none: 2
Connections:
- net labels added: RX_IN, RX_OUT, TX_IN, TX_OUT
- net labels removed: Vin
- wire segments 30 -> 61
Other:
- moved on the sheet: J1
